File: Hardware/BuggyBot KiCAD/CM5_HighSpeed.kicad_sch (KiCad schematic)
At the start: 19 parts, among them J10 690-019-298-412, J12 USB3_A, J16 Conn_01x22_Female, J22 690-019-298-412, J5 Conn_01x22_Female, J6 THD-02-R, U12 RT9742SNGV, U6 AP22653W6

Commit message: Removed all unnecessary components and modified PCB
Parts:
- removed J10: 690-019-298-412, CM5IO:EDAC 690-019-298-412, symbol CM5IO:HDMI_A_1.4
- removed J16: Conn_01x22_Female, CM5IO:Hirose_FH12-22S-0.5SH_1x22-1MP_P0.50mm_Horizontal, symbol Connector:Conn_01x22_Socket
- removed J6: THD-02-R, Connector_PinHeader_2.54mm:PinHeader_2x02_P2.54mm_Vertical, symbol Connector_Generic:Conn_02x02_Odd_Even
- removed R6, R7, R8: 2.2K 1%, Resistor_SMD:R_0402_1005Metric, symbol Device:R
Connections:
- net DPHY1_C_N: no longer names the net of Module1.187 (MIPI1_C_N)
- net DPHY1_C_P: no longer names the net of Module1.189 (MIPI1_C_P)
- net DPHY1_D0_N: no longer names the net of Module1.175 (MIPI1_D0_N)
- net DPHY1_D0_P: no longer names the net of Module1.177 (MIPI1_D0_P)
- net DPHY1_D1_N: no longer names the net of Module1.181 (MIPI1_D1_N)
- net DPHY1_D1_P: no longer names the net of Module1.183 (MIPI1_D1_P)
- net DPHY1_D2_N: no longer names the net of Module1.193 (MIPI1_D2_N)
- net DPHY1_D2_P: no longer names the net of Module1.195 (MIPI1_D2_P)
- net DPHY1_D3_N: no longer names the net of Module1.194 (MIPI1_D3_N)
- net DPHY1_D3_P: no longer names the net of Module1.196 (MIPI1_D3_P)
- net HDMI1_CEC: no longer names the net of Module1.149 (HDMI1_CEC)
- net HDMI1_CK_N: no longer names the net of Module1.166 (HDMI1_CLK_N)
- net HDMI1_CK_P: no longer names the net of Module1.164 (HDMI1_CLK_P)
- net HDMI1_D0_N: no longer names the net of Module1.160 (HDMI1_TX0_N)
- net HDMI1_D0_P: no longer names the net of Module1.158 (HDMI1_TX0_P)
- net HDMI1_D1_N: no longer names the net of Module1.154 (HDMI1_TX1_N)
- net HDMI1_D1_P: no longer names the net of Module1.152 (HDMI1_TX1_P)
- net HDMI1_D2_N: no longer names the net of Module1.148 (HDMI1_TX2_N)
- net HDMI1_D2_P: no longer names the net of Module1.146 (HDMI1_TX2_P)
- net HDMI1_HOTPLUG: no longer names the net of Module1.143 (HDMI1_HOTPLUG)
- net HDMI1_SCL: no longer names the net of Module1.147 (HDMI1_SCL)
- net HDMI1_SDA: no longer names the net of Module1.145 (HDMI1_SDA)
- no-connect marks 4 -> 24
Other:
- note added: "CAM / DISP 1 removed on 10/12/26 No-connect flags were added to CM5 pins previously connected"
- note added: "Jumpers deleted since CAM / DISP 1 removed. 10/12/26"
- note added: "Second HDMI port removed. No-connect flags were added to all CM5 pins that were previously connected to HDMI1. 10/12/26"
- note removed: "Jumpers to be fitted if DPHY1 is used"
