File: Hardware/BuggyBot KiCAD/CM5IO.kicad_pcb (KiCad board)
At the start: 4 copper layers, 160 x 90 mm, 74 parts, among them J1 Bus_M.2_Socket_M_2230_BuggyBot, J10 690-019-298-412, J11 USB_C_Receptacle_USB2.0, J12 USB3_A, J14 JST_SHBM04B-SRSS-TB, J16 Conn_01x22_Female, J2 Conn_02x07_Odd_Even, J22 690-019-298-412, J3 Conn_01x03, J5 Conn_01x22_Female, J6 THD-02-R, J8 THD-20-R, J9 THD-02-R, SW1 Right angle Tact button, U1 TPD4EUSB30, U12 RT9742SNGV, U2 TPD4EUSB30, U3 MagJack-A70-112-331N126, U6 AP22653W6, U7 ASEK-32.768KHZ-L-R-T, U8 AP3441SHE-7B

Commit message: Removed all unnecessary components and modified PCB
Parts:
- removed J10: 690-019-298-412, CM5IO:EDAC 690-019-298-412
- removed J16: Conn_01x22_Female, CM5IO:Hirose_FH12-22S-0.5SH_1x22-1MP_P0.50mm_Horizontal
- removed J3: Conn_01x03, Connector_PinHeader_2.54mm:PinHeader_1x03_P2.54mm_Vertical
- removed J6, J9: THD-02-R, Connector_PinHeader_2.54mm:PinHeader_2x02_P2.54mm_Vertical
- removed R6, R7, R8: 2.2K 1%, Resistor_SMD:R_0402_1005Metric
Connections:
- Module1 pad 143: /CM5_HighSpeed/HDMI1_HOTPLUG -> unconnected-(Module1B-HDMI1_HOTPLUG-Pad143)
- Module1 pad 145: /CM5_HighSpeed/HDMI1_SDA -> unconnected-(Module1B-HDMI1_SDA-Pad145)
- Module1 pad 146: /CM5_HighSpeed/HDMI1_D2_P -> unconnected-(Module1B-HDMI1_TX2_P-Pad146)
- Module1 pad 147: /CM5_HighSpeed/HDMI1_SCL -> unconnected-(Module1B-HDMI1_SCL-Pad147)
- Module1 pad 148: /CM5_HighSpeed/HDMI1_D2_N -> unconnected-(Module1B-HDMI1_TX2_N-Pad148)
- Module1 pad 149: /CM5_HighSpeed/HDMI1_CEC -> unconnected-(Module1B-HDMI1_CEC-Pad149)
- Module1 pad 152: /CM5_HighSpeed/HDMI1_D1_P -> unconnected-(Module1B-HDMI1_TX1_P-Pad152)
- Module1 pad 154: /CM5_HighSpeed/HDMI1_D1_N -> unconnected-(Module1B-HDMI1_TX1_N-Pad154)
- Module1 pad 158: /CM5_HighSpeed/HDMI1_D0_P -> unconnected-(Module1B-HDMI1_TX0_P-Pad158)
- Module1 pad 160: /CM5_HighSpeed/HDMI1_D0_N -> unconnected-(Module1B-HDMI1_TX0_N-Pad160)
- Module1 pad 164: /CM5_HighSpeed/HDMI1_CK_P -> unconnected-(Module1B-HDMI1_CLK_P-Pad164)
- Module1 pad 166: /CM5_HighSpeed/HDMI1_CK_N -> unconnected-(Module1B-HDMI1_CLK_N-Pad166)
- Module1 pad 175: /CM5_HighSpeed/DPHY1_D0_N -> unconnected-(Module1B-MIPI1_D0_N-Pad175)
- Module1 pad 177: /CM5_HighSpeed/DPHY1_D0_P -> unconnected-(Module1B-MIPI1_D0_P-Pad177)
- Module1 pad 181: /CM5_HighSpeed/DPHY1_D1_N -> unconnected-(Module1B-MIPI1_D1_N-Pad181)
- Module1 pad 183: /CM5_HighSpeed/DPHY1_D1_P -> unconnected-(Module1B-MIPI1_D1_P-Pad183)
- Module1 pad 187: /CM5_HighSpeed/DPHY1_C_N -> unconnected-(Module1B-MIPI1_C_N-Pad187)
- Module1 pad 189: /CM5_HighSpeed/DPHY1_C_P -> unconnected-(Module1B-MIPI1_C_P-Pad189)
- Module1 pad 193: /CM5_HighSpeed/DPHY1_D2_N -> unconnected-(Module1B-MIPI1_D2_N-Pad193)
- Module1 pad 194: /CM5_HighSpeed/DPHY1_D3_N -> unconnected-(Module1B-MIPI1_D3_N-Pad194)
- Module1 pad 195: /CM5_HighSpeed/DPHY1_D2_P -> unconnected-(Module1B-MIPI1_D2_P-Pad195)
- Module1 pad 196: /CM5_HighSpeed/DPHY1_D3_P -> unconnected-(Module1B-MIPI1_D3_P-Pad196)
- Module1 pad 57: /CM5_GPIO ( Ethernet, GPIO, SDCARD)/SD_CLK -> unconnected-(Module1A-SD_CLK-Pad57)
- Module1 pad 61: /CM5_GPIO ( Ethernet, GPIO, SDCARD)/SD_DAT3 -> unconnected-(Module1A-SD_DAT3-Pad61)
- Module1 pad 62: /CM5_GPIO ( Ethernet, GPIO, SDCARD)/SD_CMD -> unconnected-(Module1A-SD_CMD-Pad62)
- Module1 pad 63: /CM5_GPIO ( Ethernet, GPIO, SDCARD)/SD_DAT0 -> unconnected-(Module1A-SD_DAT0-Pad63)
- Module1 pad 67: /CM5_GPIO ( Ethernet, GPIO, SDCARD)/SD_DAT1 -> unconnected-(Module1A-SD_DAT1-Pad67)
- Module1 pad 69: /CM5_GPIO ( Ethernet, GPIO, SDCARD)/SD_DAT2 -> unconnected-(Module1A-SD_DAT2-Pad69)
- Module1 pad 75: /CM5_GPIO ( Ethernet, GPIO, SDCARD)/SD_PWR_ON -> unconnected-(Module1A-SD_PWR_ON-Pad75)
- Module1 pad 89: /CM5_GPIO ( Ethernet, GPIO, SDCARD)/WL_nDis -> unconnected-(Module1A-WiFi_nDisable-Pad89)
- Module1 pad 91: /CM5_GPIO ( Ethernet, GPIO, SDCARD)/BT_nDis -> unconnected-(Module1A-BT_nDisable-Pad91)
- U3 pad 11: /CM5_GPIO ( Ethernet, GPIO, SDCARD)/TR0_TAP -> unconnected-(U3-VC1-Pad11)
- U3 pad 12: /CM5_GPIO ( Ethernet, GPIO, SDCARD)/TR1_TAP -> unconnected-(U3-VC2-Pad12)
- U3 pad 13: /CM5_GPIO ( Ethernet, GPIO, SDCARD)/TR2_TAP -> unconnected-(U3-VC3-Pad13)
- U3 pad 14: /CM5_GPIO ( Ethernet, GPIO, SDCARD)/TR3_TAP -> unconnected-(U3-VC4-Pad14)
Routing:
- net /CM5_GPIO ( Ethernet, GPIO, SDCARD)/GPIO_VREF: track 103.9 -> 12.0 mm
- net /CM5_HighSpeed/HDMI1_HOTPLUG: track 81.3 -> 0.00 mm, vias 2 -> 0
- net /CM5_HighSpeed/HDMI1_SDA: track 79.5 -> 0.00 mm, vias 2 -> 0
- net /CM5_HighSpeed/HDMI1_SCL: track 78.8 -> 0.00 mm, vias 2 -> 0
- net /CM5_HighSpeed/HDMI1_CEC: track 77.7 -> 0.00 mm, vias 2 -> 0
- net /CM5_GPIO ( Ethernet, GPIO, SDCARD)/SD_CMD: track 75.2 -> 0.00 mm, vias 2 -> 0
- net /CM5_GPIO ( Ethernet, GPIO, SDCARD)/SD_DAT2: track 73.6 -> 0.00 mm
- net /CM5_HighSpeed/HDMI1_CK_N: track 73.4 -> 0.00 mm
- net /CM5_HighSpeed/HDMI1_CK_P: track 73.4 -> 0.00 mm
- net /CM5_GPIO ( Ethernet, GPIO, SDCARD)/SD_DAT3: track 72.5 -> 0.00 mm
- net /CM5_GPIO ( Ethernet, GPIO, SDCARD)/TR2_TAP: track 72.4 -> 0.00 mm
- net /CM5_HighSpeed/HDMI1_D0_N: track 71.5 -> 0.00 mm
- net /CM5_HighSpeed/HDMI1_D0_P: track 71.4 -> 0.00 mm
- net /CM5_GPIO ( Ethernet, GPIO, SDCARD)/SD_DAT1: track 71.3 -> 0.00 mm, vias 2 -> 0
- net /CM5_GPIO ( Ethernet, GPIO, SDCARD)/SD_DAT0: track 69.8 -> 0.00 mm, vias 2 -> 0
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Other:
- board text removed: "CAM/DISP 1"
- board text removed: "Fit two jumpers for CAM/DISP 1"
- board text removed: "HDMI1"
- board text removed: "J16"
- board text removed: "J3 : nBT_Dis GND"
- board text removed: "NB SD card only used for CM5 modules without eMMC"
- board text removed: "POE"
- board text removed: "SD card"
- board text removed: "nWireless_Dis"

Commit message: Added quick connect port for IMU
Parts:
- added J3: IMU Connector, Connector_JST:JST_SH_SM04B-SRSS-TB_1x04-1MP_P1.00mm_Horizontal, F.Cu at (83.0, 92.7)
Connections:
- net /CM5_HighSpeed/SCL0 renamed /CM5_GPIO ( Ethernet, GPIO, SDCARD)/SCL0
- net /CM5_HighSpeed/SDA0 renamed /CM5_GPIO ( Ethernet, GPIO, SDCARD)/SDA0
Routing:
- net /CM5_GPIO ( Ethernet, GPIO, SDCARD)/SCL0: track 108.7 -> 134.0 mm, vias 2 -> 4
- net /CM5_GPIO ( Ethernet, GPIO, SDCARD)/SDA0: track 108.1 -> 132.9 mm, vias 2 -> 4
- net /+3.3v: track 328.0 -> 330.2 mm, vias 10 -> 11

Commit message: Added connection port for LCD
Parts:
- added J4: LCD Connector, Connector_JST:JST_PH_S4B-PH-K_1x04_P2.00mm_Horizontal, F.Cu at (86.2, 93.7)
- moved J3 5.51 mm to (82.8, 87.2)
Routing:
- net /CM5_GPIO ( Ethernet, GPIO, SDCARD)/SDA0: track 132.9 -> 146.9 mm
- net /CM5_GPIO ( Ethernet, GPIO, SDCARD)/SCL0: track 134.0 -> 143.5 mm
- net /+3.3v: track 330.2 -> 334.3 mm, vias 11 -> 12

Commit message: Updated KiCad files
Parts:
- removed H6: MountingHole, CM5IO:MountingHole_2.7mm_M2.5_DIN965
- J4: footprint Connector_JST:JST_PH_S4B-PH-K_1x04_P2.00mm_Horizontal -> Connector_JST:JST_SH_SM04B-SRSS-TB_1x04-1MP_P1.00mm_Horizontal
- moved J4 4.00 mm to (82.7, 95.6)
- moved J1 0.08 mm to (226.5, 152.5)
Connections:
- J4 pad 1: /+3.3v -> GND
- J4 pad 2: GND -> /+3.3v
- J4 pad 3: /CM5_GPIO ( Ethernet, GPIO, SDCARD)/SCL0 -> /CM5_GPIO ( Ethernet, GPIO, SDCARD)/SDA0
- J4 pad 4: /CM5_GPIO ( Ethernet, GPIO, SDCARD)/SDA0 -> /CM5_GPIO ( Ethernet, GPIO, SDCARD)/SCL0
Routing:
- net /+3.3v: track 334.3 -> 336.4 mm
- net /CM5_GPIO ( Ethernet, GPIO, SDCARD)/SDA0: track 146.9 -> 148.1 mm
