File: Hardware/BuggyBot KiCAD/CM5IO.kicad_pcb (KiCad board)
At the start: 4 copper layers, 160 x 90 mm, 67 parts, among them J1 Bus_M.2_Socket_M_2230_BuggyBot, J11 USB_C_Receptacle_USB2.0, J12 USB3_A, J14 JST_SHBM04B-SRSS-TB, J2 Conn_02x07_Odd_Even, J22 690-019-298-412, J3 IMU Connector, J4 LCD Connector, J5 Conn_01x22_Female, J8 THD-20-R, SW1 Right angle Tact button, U1 TPD4EUSB30, U12 RT9742SNGV, U2 TPD4EUSB30, U3 MagJack-A70-112-331N126, U6 AP22653W6, U7 ASEK-32.768KHZ-L-R-T, U8 AP3441SHE-7B

Commit message: Updated KiCad files and added redesign pcb file
Parts:
- added J6: Line Sensor, Connector_JST:JST_SH_SM04B-SRSS-TB_1x04-1MP_P1.00mm_Horizontal, F.Cu at (65.7, 106.3)
- added J7: Line Sensor, Connector_JST:JST_SH_SM04B-SRSS-TB_1x04-1MP_P1.00mm_Horizontal, F.Cu at (65.7, 113.9)

Commit message: Updated KiCad files
Parts:
- removed H7, H8: MountingHole, CM5IO:MountingHole_2.7mm_M2.5_DIN965
- added H6: MountingHole, CM5IO:MountingHole_2.7mm_M2.5_DIN965, F.Cu at (145.7, 133.4)
- moved H2 179.3 mm to (240.5, 71.7)
- moved J3 157.9 mm to (233.8, 133.3), turned to 0 degrees
- moved J7 153.6 mm to (218.0, 133.3)
- moved J4 148.1 mm to (225.9, 133.3), turned to 0 degrees
- moved J6 147.0 mm to (210.2, 133.3)
- moved H4 102.7 mm to (240.5, 133.3)
- moved SW1 94.8 mm to (201.0, 72.0)
- moved D3 90.9 mm to (234.1, 70.8), turned to 0 degrees
- moved R17 86.3 mm to (232.9, 72.9), turned to -90 degrees
- moved TP1 86.1 mm to (233.9, 73.3), turned to 180 degrees
- moved H1 82.0 mm to (106.5, 71.7)
- moved U3 77.7 mm to (113.7, 83.5), turned to -90 degrees
- moved J1 76.2 mm to (219.5, 76.6), turned to 0 degrees
- moved J12 76.1 mm to (112.7, 103.7), turned to -90 degrees
- moved H5 68.3 mm to (203.7, 133.4)
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Connections:
- J3 pad 3: /CM5_GPIO ( Ethernet, GPIO, SDCARD)/SDA0 -> /CM5_GPIO ( Ethernet, GPIO, SDCARD)/GPIO2
- J3 pad 4: /CM5_GPIO ( Ethernet, GPIO, SDCARD)/SCL0 -> /CM5_GPIO ( Ethernet, GPIO, SDCARD)/GPIO3
- J4 pad 3: /CM5_GPIO ( Ethernet, GPIO, SDCARD)/SDA0 -> /CM5_GPIO ( Ethernet, GPIO, SDCARD)/GPIO2
- J4 pad 4: /CM5_GPIO ( Ethernet, GPIO, SDCARD)/SCL0 -> /CM5_GPIO ( Ethernet, GPIO, SDCARD)/GPIO3
- J5 pad 20: /CM5_GPIO ( Ethernet, GPIO, SDCARD)/SCL0 -> /CM5_HighSpeed/SCL0
- J5 pad 21: /CM5_GPIO ( Ethernet, GPIO, SDCARD)/SDA0 -> /CM5_HighSpeed/SDA0
- Module1 pad 80: /CM5_GPIO ( Ethernet, GPIO, SDCARD)/SCL0 -> /CM5_HighSpeed/SCL0
- Module1 pad 82: /CM5_GPIO ( Ethernet, GPIO, SDCARD)/SDA0 -> /CM5_HighSpeed/SDA0
Routing:
- net GND: track 733.5 -> 206.2 mm, vias 447 -> 136
- net /+3.3v: track 336.4 -> 172.7 mm, vias 12 -> 2
- net /CM5_GPIO ( Ethernet, GPIO, SDCARD)/SDA0: track 148.1 -> 0.00 mm, vias 4 -> 0
- net /CM5_GPIO ( Ethernet, GPIO, SDCARD)/SCL0: track 143.3 -> 0.00 mm, vias 4 -> 0
- net /CM5_HighSpeed/VBUS: track 80.6 -> 176.3 mm, vias 4 -> 5
- net /CM5_GPIO ( Ethernet, GPIO, SDCARD)/PMIC_ENABLE: track 53.1 -> 136.7 mm, vias 2 -> 3
- net /CM5_GPIO ( Ethernet, GPIO, SDCARD)/CAM_GPIO1: track 113.1 -> 53.9 mm
- net /CM5_GPIO ( Ethernet, GPIO, SDCARD)/CAM_GPIO0: track 117.8 -> 60.0 mm
- net /CM5_GPIO ( Ethernet, GPIO, SDCARD)/VBAT: track 154.8 -> 103.0 mm
- net /CM5_HighSpeed/SCL0: track 0.00 -> 51.3 mm, vias 0 -> 2
- net /CM5_GPIO ( Ethernet, GPIO, SDCARD)/GPIO7: track 99.3 -> 49.5 mm, vias 1 -> 2
- net /CM5_GPIO ( Ethernet, GPIO, SDCARD)/nRPIBOOT: track 69.2 -> 119.0 mm, vias 2 -> 3
- net /CM5_HighSpeed/DPHY0_D3_N: track 92.8 -> 43.2 mm
- net /CM5_HighSpeed/DPHY0_D3_P: track 92.8 -> 43.1 mm
- net /CM5_GPIO ( Ethernet, GPIO, SDCARD)/GPIO8: track 101.5 -> 52.2 mm, vias 1 -> 2
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- removed copper zone on B.Cu, net /+5v
- removed copper zone on F.Cu, net /+5v
- removed copper zone on B.Cu, net /CM5_HighSpeed/VBUS
- removed copper zone on F.Cu, net /PCIe-M2/M2_3v3
Other:
- board size 160 x 90 mm -> 139.6 x 67.2 mm

Commit message: Updated KiCAD files
Parts:
- moved H5 2.00 mm to (203.7, 131.4)
- moved H6 2.00 mm to (145.7, 131.4)
- moved J8 2.00 mm to (150.6, 132.7)
- moved C9 1.71 mm to (233.3, 119.7)
- moved C18 1.58 mm to (233.2, 113.7)
Routing:
- net GND: track 206.2 -> 730.5 mm, vias 136 -> 137
- net /CM5_GPIO ( Ethernet, GPIO, SDCARD)/GPIO2: track 164.6 -> 84.1 mm, vias 3 -> 2
- net /+5v: track 238.6 -> 200.9 mm, vias 11 -> 18
- net /+3.3v: track 172.7 -> 195.6 mm, vias 2 -> 3
- net /CM5_GPIO ( Ethernet, GPIO, SDCARD)/GPIO21: track 67.3 -> 44.9 mm
- net /CM5_GPIO ( Ethernet, GPIO, SDCARD)/GPIO20: track 63.0 -> 43.6 mm
- net (no net): track 0.00 -> 9.80 mm
- net /CM5_GPIO ( Ethernet, GPIO, SDCARD)/ID_SC: track 51.1 -> 47.9 mm
- net /CM5_GPIO ( Ethernet, GPIO, SDCARD)/GPIO6: track 48.6 -> 45.7 mm
- net /CM5_GPIO ( Ethernet, GPIO, SDCARD)/GPIO24: track 60.5 -> 58.1 mm
- net /CM5_GPIO ( Ethernet, GPIO, SDCARD)/GPIO19: track 45.9 -> 43.5 mm
- net /CM5_GPIO ( Ethernet, GPIO, SDCARD)/GPIO3: track 153.4 -> 151.4 mm
- net /CM5_GPIO ( Ethernet, GPIO, SDCARD)/GPIO23: track 60.1 -> 58.1 mm
- net /CM5_GPIO ( Ethernet, GPIO, SDCARD)/GPIO11: track 51.1 -> 49.1 mm
- net /CM5_GPIO ( Ethernet, GPIO, SDCARD)/GPIO22: track 61.0 -> 59.0 mm
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- added copper zone on B.Cu, net /+5v
- added copper zone on F.Cu, net /+5v
Other:
- board text added: "J8"

Commit message: Update BuggyBot KiCad project
Parts:
- added H7: MountingHole, CM5IO:MountingHole_2.7mm_M2.5_DIN965, F.Cu at (136.3, 72.5)
- moved R11 0.18 mm to (206.2, 87.9)
Routing:
- net /+3.3v: track 195.6 -> 345.3 mm, vias 3 -> 7
- net /PCIe-M2/M2_3v3: track 68.2 -> 209.8 mm
- net /CM5_GPIO ( Ethernet, GPIO, SDCARD)/GPIO2: track 84.1 -> 159.6 mm, vias 2 -> 4
- net /+5v: track 200.9 -> 243.8 mm, vias 18 -> 19
- net /CM5_GPIO ( Ethernet, GPIO, SDCARD)/GPIO21: track 44.9 -> 64.9 mm
- net GND: track 730.5 -> 750.0 mm, vias 137 -> 146
- net /CM5_GPIO ( Ethernet, GPIO, SDCARD)/GPIO20: track 43.6 -> 61.1 mm
- net (no net): track 9.80 -> 0.00 mm
- net /CM5_GPIO ( Ethernet, GPIO, SDCARD)/GPIO3: track 151.4 -> 154.5 mm
- net /CM5_HighSpeed/VBUS: track 176.3 -> 178.3 mm
- net /CM5_HighSpeed/USB3-0-D_P: track 73.4 -> 74.5 mm
- net /CM5_HighSpeed/USB3-0-D_N: track 73.4 -> 74.6 mm
- net /CM5_HighSpeed/USB3-0-TX_N: track 82.3 -> 83.3 mm
- net /CM5_HighSpeed/USB3-0-TX_P: track 82.9 -> 83.9 mm
- net /CM5_HighSpeed/USB3-0-RX_P: track 60.7 -> 61.6 mm
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Other:
- board text removed: "J8"
