File: Hardware/BuggyBot KiCAD/CM5IORedesign.kicad_pcb (KiCad board)
At the start: 4 copper layers, 62 parts, among them J1 Bus_M.2_Socket_M_2230_BuggyBot, J11 USB_C_Receptacle_USB2.0, J12 USB3_A, J14 JST_SHBM04B-SRSS-TB, J2 Conn_02x07_Odd_Even, J22 690-019-298-412, J3 IMU Connector, J4 LCD Connector, J5 Conn_01x22_Female, J6 Line Sensor, J7 Line Sensor, J8 THD-20-R, SW1 Right angle Tact button, U1 TPD4EUSB30, U12 RT9742SNGV, U2 TPD4EUSB30, U3 MagJack-A70-112-331N126, U6 AP22653W6, U7 ASEK-32.768KHZ-L-R-T, U8 AP3441SHE-7B

Commit message: Updated KiCAD files
Parts:
- added REF**: MountingHole_2.7mm_M2.5_DIN965, CM5IO:MountingHole_2.7mm_M2.5_DIN965, F.Cu at (240.5, 133.7)
- added REF**: MountingHole_2.7mm_M2.5_DIN965, CM5IO:MountingHole_2.7mm_M2.5_DIN965, F.Cu at (106.5, 133.7)
- added REF**: MountingHole_2.7mm_M2.5_DIN965, CM5IO:MountingHole_2.7mm_M2.5_DIN965, F.Cu at (106.5, 71.7)
- added REF**: MountingHole_2.7mm_M2.5_DIN965, CM5IO:MountingHole_2.7mm_M2.5_DIN965, F.Cu at (240.5, 71.7)
- moved J11 105.2 mm to (234.2, 115.5), turned to 90 degrees
- moved C18 100.8 mm to (226.3, 111.5), turned to 90 degrees
- moved C9 95.9 mm to (226.3, 117.5), turned to -90 degrees
- moved SW1 94.8 mm to (201.0, 74.4)
- moved C3 86.5 mm to (216.8, 115.8), turned to 180 degrees
- moved R12 81.5 mm to (211.3, 114.9), turned to -90 degrees
- moved U6 79.3 mm to (208.4, 114.2), turned to 0 degrees
- moved C2 76.9 mm to (204.9, 113.3), turned to -90 degrees
- moved J8 66.5 mm to (153.0, 131.4)
- moved J2 61.6 mm to (113.9, 130.8), turned to 180 degrees
- moved J5 58.4 mm to (148.9, 75.1)
- moved BT1 50.8 mm to (143.2, 101.5), turned to 90 degrees
- moved U3 50.1 mm to (120.0, 81.6), turned to -90 degrees
- moved C12 45.4 mm to (143.2, 122.7)
- moved C13 45.4 mm to (148.4, 121.8)
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Routing:
- net /CM5_HighSpeed/PCIE_TX_N: track 0.00 -> 117.5 mm, vias 0 -> 2
- net /CM5_HighSpeed/PCIE_TX_P: track 0.00 -> 117.5 mm, vias 0 -> 2
- net /CM5_HighSpeed/PCIE_RX_P: track 0.00 -> 113.1 mm, vias 0 -> 2
- net /CM5_HighSpeed/PCIE_RX_N: track 0.00 -> 113.0 mm, vias 0 -> 2
- net /CM5_HighSpeed/PCIE_CLK_N: track 0.00 -> 112.8 mm, vias 0 -> 2
- net /CM5_HighSpeed/PCIE_CLK_P: track 0.00 -> 112.0 mm, vias 0 -> 2
- net /CM5_HighSpeed/PCIE_PWR_EN: track 0.00 -> 101.5 mm, vias 0 -> 2
- net /CM5_HighSpeed/PCIE_nWAKE: track 0.00 -> 92.7 mm, vias 0 -> 2
- net /CM5_HighSpeed/PCIE_nCLKREQ: track 0.00 -> 90.7 mm, vias 0 -> 2
- net /CM5_HighSpeed/PCIE_nRST: track 0.00 -> 86.9 mm, vias 0 -> 2
- net /PCIe-M2/M2_3v3: track 0.00 -> 68.2 mm, vias 0 -> 3
- net /CM5_GPIO ( Ethernet, GPIO, SDCARD)/CAM_GPIO0: track 0.00 -> 54.9 mm
- net /CM5_GPIO ( Ethernet, GPIO, SDCARD)/SCL0: track 0.00 -> 48.3 mm, vias 0 -> 2
- net /CM5_GPIO ( Ethernet, GPIO, SDCARD)/CAM_GPIO1: track 0.00 -> 47.2 mm
- net /CM5_GPIO ( Ethernet, GPIO, SDCARD)/SDA0: track 0.00 -> 46.5 mm
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- added copper zone on F.Cu, net /PCIe-M2/M2_3v3
Other:
- board outline added: 139.3 x 67.6 mm

Commit message: Updated KiCad design files
Parts:
- added REF**: MountingHole_2.7mm_M2.5_DIN965, CM5IO:MountingHole_2.7mm_M2.5_DIN965, F.Cu at (203.7, 133.4)
- added REF**: MountingHole_2.7mm_M2.5_DIN965, CM5IO:MountingHole_2.7mm_M2.5_DIN965, F.Cu at (145.7, 133.4)
- moved J7 24.7 mm to (210.2, 133.3)
- moved J3 24.0 mm to (233.8, 133.3)
- moved J6 9.66 mm to (218.0, 133.3)
- moved J4 8.54 mm to (225.9, 133.3)
- moved J22 7.45 mm to (126.8, 126.8)
- moved D1 7.43 mm to (137.5, 135.1)
- moved R1 7.43 mm to (140.6, 132.6)
- moved C12 7.43 mm to (136.3, 125.7)
- moved C13 7.43 mm to (141.6, 124.8)
- moved D2 7.43 mm to (141.1, 135.1)
- moved R10 7.43 mm to (138.4, 132.6)
- moved TP3 7.43 mm to (141.2, 132.3)
- moved TP5 7.43 mm to (137.9, 132.3)
- moved U12 7.43 mm to (138.9, 123.8)
- moved R3 6.57 mm to (126.0, 90.8)
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Routing:
- net /CM5_GPIO ( Ethernet, GPIO, SDCARD)/nPWR_LED: track 0.00 -> 91.1 mm, vias 0 -> 2
- net Net-(Module1A-LED_nACT): track 0.00 -> 69.5 mm, vias 0 -> 2
- net /CM5_HighSpeed/HDMI0_SDA: track 1.63 -> 62.1 mm
- net /CM5_HighSpeed/HDMI0_SCL: track 0.00 -> 58.5 mm
- net /CM5_HighSpeed/HDMI0_CK_N: track 0.00 -> 55.7 mm
- net /CM5_HighSpeed/HDMI0_HOTPLUG: track 0.00 -> 55.6 mm, vias 0 -> 2
- net /CM5_HighSpeed/HDMI0_CK_P: track 0.00 -> 55.5 mm
- net /CM5_HighSpeed/HDMI0_D0_N: track 0.00 -> 53.0 mm
- net /CM5_HighSpeed/HDMI0_D0_P: track 0.00 -> 52.9 mm
- net /CM5_HighSpeed/HDMI0_CEC: track 0.00 -> 52.8 mm, vias 0 -> 2
- net /CM5_HighSpeed/HDMI0_D1_N: track 0.00 -> 50.4 mm
- net /CM5_HighSpeed/HDMI0_D1_P: track 0.00 -> 50.3 mm
- net /CM5_HighSpeed/HDMI0_D2_P: track 0.00 -> 48.0 mm
- net /CM5_HighSpeed/HDMI0_D2_N: track 0.00 -> 47.9 mm
- net Net-(U3-LEDY_K): track 0.00 -> 31.9 mm
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Other:
- board size 139.3 x 67.6 mm -> 139.6 x 67.2 mm

Commit message: Updated BuggyBot KiCad project
Parts:
- moved BT1 96.7 mm to (41.2, 90.0)
Routing:
- net /CM5_GPIO ( Ethernet, GPIO, SDCARD)/TRD3_N: track 0.00 -> 102.3 mm
- net /CM5_GPIO ( Ethernet, GPIO, SDCARD)/TRD3_P: track 0.00 -> 102.2 mm
- net /CM5_GPIO ( Ethernet, GPIO, SDCARD)/ETH_LEDG: track 0.00 -> 99.3 mm, vias 0 -> 2
- net /CM5_GPIO ( Ethernet, GPIO, SDCARD)/TRD1_P: track 0.00 -> 94.9 mm
- net /CM5_GPIO ( Ethernet, GPIO, SDCARD)/ETH_LEDY: track 0.00 -> 94.1 mm, vias 0 -> 2
- net /CM5_GPIO ( Ethernet, GPIO, SDCARD)/TRD2_N: track 7.93 -> 100.1 mm
- net /CM5_GPIO ( Ethernet, GPIO, SDCARD)/TRD2_P: track 8.07 -> 99.9 mm
- net /CM5_GPIO ( Ethernet, GPIO, SDCARD)/TRD0_P: track 0.00 -> 90.7 mm
- net /CM5_GPIO ( Ethernet, GPIO, SDCARD)/TRD1_N: track 9.57 -> 95.1 mm
- net /CM5_GPIO ( Ethernet, GPIO, SDCARD)/TRD0_N: track 5.75 -> 90.7 mm
- net /CM5_HighSpeed/USB3-0-TX_P: track 0.00 -> 84.6 mm, vias 0 -> 1
- net /CM5_HighSpeed/USB3-0-TX_N: track 0.00 -> 84.6 mm, vias 0 -> 1
- net /CM5_HighSpeed/USB3-0-D_N: track 0.00 -> 73.2 mm, vias 0 -> 2
- net /CM5_HighSpeed/USB3-0-D_P: track 0.00 -> 73.1 mm, vias 0 -> 2
- net /CM5_HighSpeed/USB3-0-RX_N: track 0.00 -> 59.9 mm, vias 0 -> 2
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
Commit message: Updated KiCad files
Parts:
- moved BT1 97.2 mm to (137.5, 103.0)
- moved R11 1.62 mm to (206.4, 87.9)
Routing:
- net /CM5_GPIO ( Ethernet, GPIO, SDCARD)/PWR_BUT: track 0.00 -> 129.9 mm, vias 0 -> 4
- net /CM5_GPIO ( Ethernet, GPIO, SDCARD)/PMIC_ENABLE: track 0.00 -> 122.4 mm, vias 0 -> 3
- net /CM5_GPIO ( Ethernet, GPIO, SDCARD)/nRPIBOOT: track 0.00 -> 112.1 mm, vias 0 -> 3
- net /CM5_GPIO ( Ethernet, GPIO, SDCARD)/EEPROM_nWP: track 0.00 -> 98.5 mm, vias 0 -> 3
- net /CM5_GPIO ( Ethernet, GPIO, SDCARD)/SYNC_OUT: track 0.00 -> 98.0 mm, vias 0 -> 3
- net /USB2_P: track 0.00 -> 83.7 mm, vias 0 -> 2
- net /USB2_N: track 0.00 -> 83.6 mm, vias 0 -> 2
- net /CC1: track 0.00 -> 80.7 mm, vias 0 -> 2
- net /CM5_GPIO ( Ethernet, GPIO, SDCARD)/USBOTG: track 0.00 -> 71.0 mm, vias 0 -> 1
- net /CC2: track 0.00 -> 64.6 mm, vias 0 -> 2
- net /CM5_HighSpeed/DPHY0_C_N: track 0.00 -> 47.1 mm, vias 0 -> 2
- net /CM5_HighSpeed/DPHY0_C_P: track 0.00 -> 47.1 mm, vias 0 -> 2
- net /CM5_HighSpeed/DPHY0_D2_N: track 0.00 -> 44.8 mm, vias 0 -> 2
- net /CM5_HighSpeed/DPHY0_D2_P: track 0.00 -> 44.8 mm, vias 0 -> 2
- net /CM5_HighSpeed/DPHY0_D3_N: track 0.00 -> 43.2 mm, vias 0 -> 2
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