File: Hardware/BuggyBot KiCAD/CM5IO.kicad_sch (KiCad schematic)
At the start: 12 parts, among them J11 USB_C_Receptacle_USB2.0

Commit message: Removed all unnecessary components and modified PCB
Connections:
- no-connect marks 2 -> 5
Other:
- sheet CM5_HighSpeed ports: added none; removed GPIO_VREF, ID_SC, ID_SD
Changed lines of the file:
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@@
+	)
+	(no_connect
+		(at 180.34 96.52)
+	)
+	(no_connect
+		(at 149.86 96.52)
+	)
+	(no_connect
+		(at 146.05 96.52)
 	)
 	(no_connect
@@
 			)
 		)
-		(pin "ID_SC" input
-			(at 149.86 96.52 270)
-			(effects
-				(font
-					(size 1.27 1.27)
-				)
-				(justify left)
-			)
-		)
-		(pin "ID_SD" input
-			(at 146.05 96.52 270)
-			(effects
-				(font
-					(size 1.27 1.27)
-				)
-				(justify left)
-			)
-		)
 		(pin "SCL0" input
 			(at 138.43 96.52 270)
@@
 			(effects
 				(font
-					(size 1.27 1.27)
-				)
-				(justify left)
-			)
-		)
-		(pin "GPIO_VREF" input
-			(at 180.34 96.52 270)
-			(effects
-				(font

Commit message: Updated KiCad files
Parts:
- removed H6: MountingHole, CM5IO:MountingHole_2.7mm_M2.5_DIN965, symbol Mechanical:MountingHole
Changed lines of the file:
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@@
-	)
-	(symbol
-		(lib_id "Mechanical:MountingHole")
-		(at 43.815 170.815 0)
-		(unit 1)
-		(body_style 1)
-		(exclude_from_sim yes)
-		(in_bom no)
-		(on_board yes)
-		(in_pos_files yes)
-		(dnp yes)
-		(property "Reference" "H6"
-			(at 46.355 169.672 0)
-			(show_name no)
-			(do_not_autoplace no)
-			(effects
-				(font
-					(size 1.27 1.27)
-				)
-				(justify left)
-			)
-		)
-		(property "Value" "MountingHole"
-			(at 46.355 171.958 0)
-			(show_name no)
-			(do_not_autoplace no)
-			(effects
-				(font
-					(size 1.27 1.27)
-				)
-				(justify left)
-			)
-		)
-		(property "Footprint" "CM5IO:MountingHole_2.7mm_M2.5_DIN965"
-			(at 43.815 170.815 0)
-			(hide yes)
-			(show_name no)
-			(do_not_autoplace no)
-			(effects
-				(font
-					(size 1.27 1.27)
-				)
-			)
-		)
-		(property "Datasheet" ""
-			(at 43.815 170.815 0)
-			(hide yes)
-			(show_name no)
-			(do_not_autoplace no)
-			(effects
-				(font
-					(size 1.27 1.27)
-				)
-			)
-		)
-		(property "Description" ""
-			(at 43.815 170.815 0)
-			(hide yes)
-			(show_name no)
-			(do_not_autoplace no)
-			(effects
-				(font
-					(size 1.27 1.27)
-				)
-			)
-		)
-		(property "Field4" "nf"
-			(at 43.815 170.815 0)
-			(hide yes)
-			(show_name no)
-			(do_not_autoplace no)
-			(effects
-				(font
-					(size 1.27 1.27)
-				)
-			)
-		)
-		(property "Field5" "nf"
-			(at 43.815 170.815 0)
-			(hide yes)
-			(show_name no)
-			(do_not_autoplace no)
-			(effects
-				(font
-					(size 1.27 1.27)
-				)
-			)
-		)
-		(property "Field6" "nf"
-			(at 43.815 170.815 0)
-			(hide yes)
-			(show_name no)
-			(do_not_autoplace no)
-			(effects
-				(font
-					(size 1.27 1.27)
-				)
-			)
-		)
-		(property "Field7" "nf"
-			(at 43.815 170.815 0)
-			(hide yes)
-			(show_name no)
-			(do_not_autoplace no)
-			(effects
-				(font
-					(size 1.27 1.27)
-				)
-			)
-		)
-		(property "Part Description" "M2.5 mounting hole"
-			(at 43.815 170.815 0)
-			(hide yes)
-			(show_name no)
-			(do_not_autoplace no)
-			(effects
-				(font
-					(size 1.27 1.27)
-				)
-			)
-		)
-		(instances
-			(project "CM5IO"
-				(path "/e63e39d7-6ac0-4ffd-8aa3-1841a4541b55"
-					(reference "H6")
-					(unit 1)
-				)
-			)
-		)
 	)
 	(symbol

Commit message: Updated KiCad files and added redesign pcb file
Other:
- moved on the sheet: H8
Changed lines of the file:
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@@
 	(symbol
 		(lib_id "Mechanical:MountingHole")
-		(at 43.815 180.975 0)
+		(at 43.18 187.96 0)
 		(unit 1)
 		(body_style 1)
@@
 		(dnp yes)
 		(property "Reference" "H8"
-			(at 46.355 179.832 0)
+			(at 45.72 186.817 0)
 			(show_name no)
 			(do_not_autoplace no)
@@
 		)
 		(property "Value" "MountingHole"
-			(at 46.355 182.118 0)
+			(at 45.72 189.103 0)
 			(show_name no)
 			(do_not_autoplace no)
@@
 		)
 		(property "Footprint" "CM5IO:MountingHole_2.7mm_M2.5_DIN965"
-			(at 43.815 180.975 0)
+			(at 43.18 187.96 0)
 			(hide yes)
 			(show_name no)
@@
 		)
 		(property "Datasheet" ""
-			(at 43.815 180.975 0)
+			(at 43.18 187.96 0)
 			(hide yes)
 			(show_name no)
@@
 		)
 		(property "Description" ""
-			(at 43.815 180.975 0)
+			(at 43.18 187.96 0)
 			(hide yes)
 			(show_name no)
@@
 		)
 		(property "Field4" "nf"
-			(at 43.815 180.975 0)
+			(at 43.18 187.96 0)
 			(hide yes)
 			(show_name no)
@@
 		)
 		(property "Field5" "nf"
-			(at 43.815 180.975 0)
+			(at 43.18 187.96 0)
 			(hide yes)
 			(show_name no)
@@
 		)
 		(property "Field6" "nf"
-			(at 43.815 180.975 0)
+			(at 43.18 187.96 0)
 			(hide yes)
 			(show_name no)
@@
 		)
 		(property "Field7" "nf"
-			(at 43.815 180.975 0)
+			(at 43.18 187.96 0)
 			(hide yes)
 			(show_name no)
@@
 		)
 		(property "Part Description" "M2.5 mounting hole"
-			(at 43.815 180.975 0)
+			(at 43.18 187.96 0)
 			(hide yes)
 			(show_name no)

Commit message: Updated KiCAD files
Parts:
- added H6: MountingHole, CM5IO:MountingHole_2.7mm_M2.5_DIN965, symbol Mechanical:MountingHole
Other:
- moved on the sheet: H5, H7, H8
Changed lines of the file:
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@@
 	(symbol
 		(lib_id "Mechanical:MountingHole")
-		(at 43.815 165.735 0)
+		(at 43.18 166.37 0)
 		(unit 1)
 		(body_style 1)
@@
 		(dnp yes)
 		(property "Reference" "H5"
-			(at 46.355 164.592 0)
+			(at 45.72 165.227 0)
 			(show_name no)
 			(do_not_autoplace no)
@@
 		)
 		(property "Value" "MountingHole"
-			(at 46.355 166.878 0)
+			(at 45.72 167.513 0)
 			(show_name no)
 			(do_not_autoplace no)
@@
 		)
 		(property "Footprint" "CM5IO:MountingHole_2.7mm_M2.5_DIN965"
-			(at 43.815 165.735 0)
+			(at 43.18 166.37 0)
 			(hide yes)
 			(show_name no)
@@
 		)
 		(property "Datasheet" ""
-			(at 43.815 165.735 0)
+			(at 43.18 166.37 0)
 			(hide yes)
 			(show_name no)
@@
 		)
 		(property "Description" ""
-			(at 43.815 165.735 0)
+			(at 43.18 166.37 0)
 			(hide yes)
 			(show_name no)
@@
 		)
 		(property "Field4" "nf"
-			(at 43.815 165.735 0)
+			(at 43.18 166.37 0)
 			(hide yes)
 			(show_name no)
@@
 		)
 		(property "Field5" "nf"
-			(at 43.815 165.735 0)
+			(at 43.18 166.37 0)
 			(hide yes)
 			(show_name no)
@@
 		)
 		(property "Field6" "nf"
-			(at 43.815 165.735 0)
+			(at 43.18 166.37 0)
 			(hide yes)
 			(show_name no)
@@
 		)
 		(property "Field7" "nf"
-			(at 43.815 165.735 0)
+			(at 43.18 166.37 0)
 			(hide yes)
 			(show_name no)
@@
 		)
 		(property "Part Description" "M2.5 mounting hole"
-			(at 43.815 165.735 0)
+			(at 43.18 166.37 0)
 			(hide yes)
 			(show_name no)
@@
 	(symbol
 		(lib_id "Mechanical:MountingHole")
-		(at 43.18 187.96 0)
+		(at 43.18 181.61 0)
 		(unit 1)
 		(body_style 1)
@@
 		(dnp yes)
 		(property "Reference" "H8"
-			(at 45.72 186.817 0)
+			(at 45.72 180.467 0)
 			(show_name no)
 			(do_not_autoplace no)
@@
 		)
 		(property "Value" "MountingHole"
-			(at 45.72 189.103 0)
+			(at 45.72 182.753 0)
 			(show_name no)
 			(do_not_autoplace no)
@@
 		)
 		(property "Footprint" "CM5IO:MountingHole_2.7mm_M2.5_DIN965"
-			(at 43.18 187.96 0)
+			(at 43.18 181.61 0)
 			(hide yes)
 			(show_name no)
@@
 		)
 		(property "Datasheet" ""
-			(at 43.18 187.96 0)
+			(at 43.18 181.61 0)
 			(hide yes)
 			(show_name no)
@@
 		)
 		(property "Description" ""
-			(at 43.18 187.96 0)
+			(at 43.18 181.61 0)
 			(hide yes)
 			(show_name no)
@@
 		)
 		(property "Field4" "nf"
-			(at 43.18 187.96 0)
+			(at 43.18 181.61 0)
 			(hide yes)
 			(show_name no)
@@
 		)
 		(property "Field5" "nf"
-			(at 43.18 187.96 0)
+			(at 43.18 181.61 0)
 			(hide yes)
 			(show_name no)
@@
 		)
 		(property "Field6" "nf"
-			(at 43.18 187.96 0)
+			(at 43.18 181.61 0)
 			(hide yes)
 			(show_name no)
@@
 		)
 		(property "Field7" "nf"
-			(at 43.18 187.96 0)
+			(at 43.18 181.61 0)
 			(hide yes)
 			(show_name no)
@@
 		)
 		(property "Part Description" "M2.5 mounting hole"
-			(at 43.18 187.96 0)
+			(at 43.18 181.61 0)
 			(hide yes)
 			(show_name no)
@@
 	(symbol
 		(lib_id "Mechanical:MountingHole")
-		(at 43.815 175.895 0)
+		(at 43.18 176.53 0)
 		(unit 1)
 		(body_style 1)
@@
 		(dnp yes)
 		(property "Reference" "H7"
-			(at 46.355 174.752 0)
+			(at 45.72 175.387 0)
 			(show_name no)
 			(do_not_autoplace no)
@@
 		)
 		(property "Value" "MountingHole"
-			(at 46.355 177.038 0)
+			(at 45.72 177.673 0)
 			(show_name no)
 			(do_not_autoplace no)
@@
 		)
 		(property "Footprint" "CM5IO:MountingHole_2.7mm_M2.5_DIN965"
-			(at 43.815 175.895 0)
+			(at 43.18 176.53 0)
 			(hide yes)
 			(show_name no)
@@
 		)
 		(property "Datasheet" ""
-			(at 43.815 175.895 0)
+			(at 43.18 176.53 0)
 			(hide yes)
 			(show_name no)
@@
 		)
 		(property "Description" ""
-			(at 43.815 175.895 0)
+			(at 43.18 176.53 0)
 			(hide yes)
 			(show_name no)
@@
 		)
 		(property "Field4" "nf"
-			(at 43.815 175.895 0)
+			(at 43.18 176.53 0)
 			(hide yes)
 			(show_name no)
@@
 		)
 		(property "Field5" "nf"
-			(at 43.815 175.895 0)
+			(at 43.18 176.53 0)
 			(hide yes)
 			(show_name no)
@@
 		)
 		(property "Field6" "nf"
-			(at 43.815 175.895 0)
+			(at 43.18 176.53 0)
 			(hide yes)
 			(show_name no)
@@
 		)
 		(property "Field7" "nf"
-			(at 43.815 175.895 0)
+			(at 43.18 176.53 0)
 			(hide yes)
 			(show_name no)
@@
 		)
 		(property "Part Description" "M2.5 mounting hole"
-			(at 43.815 175.895 0)
+			(at 43.18 176.53 0)
 			(hide yes)
 			(show_name no)
@@
 					(unit 1)
 				)
+			)
+		)
+	)
+	(symbol
+		(lib_id "Mechanical:MountingHole")
+		(at 43.18 171.45 0)
+		(unit 1)
+		(body_style 1)
+		(exclude_from_sim yes)
+		(in_bom no)
+		(on_board yes)
+		(in_pos_files yes)
+		(dnp yes)
+		(property "Reference" "H6"
+			(at 45.72 170.307 0)
+			(show_name no)
+			(do_not_autoplace no)
+			(effects
+				(font
+					(size 1.27 1.27)
+				)
+				(justify left)
+			)
+		)
+		(property "Value" "MountingHole"
+			(at 45.72 172.593 0)
+			(show_name no)
+			(do_not_autoplace no)
+			(effects
+				(font
+					(size 1.27 1.27)
+				)
+				(justify left)
+			)
+		)
+		(property "Footprint" "CM5IO:MountingHole_2.7mm_M2.5_DIN965"
+			(at 43.18 171.45 0)
+			(hide yes)
+			(show_name no)
+			(do_not_autoplace no)
+			(effects
+				(font
+					(size 1.27 1.27)
+				)
+			)
+		)
+		(property "Datasheet" ""
+			(at 43.18 171.45 0)
+			(hide yes)
+			(show_name no)
+			(do_not_autoplace no)
+			(effects
+				(font
+					(size 1.27 1.27)
+				)
+			)
+		)
+		(property "Description" ""
+			(at 43.18 171.45 0)
+			(hide yes)
+			(show_name no)
+			(do_not_autoplace no)
+			(effects
+				(font
+					(size 1.27 1.27)
+				)
+			)
+		)
+		(property "Field4" "nf"
+			(at 43.18 171.45 0)
+			(hide yes)
+			(show_name no)
+			(do_not_autoplace no)
+			(effects
+				(font
+					(size 1.27 1.27)
+				)
+			)
+		)
+		(property "Field5" "nf"
+			(at 43.18 171.45 0)
+			(hide yes)
+			(show_name no)
+			(do_not_autoplace no)
+			(effects
+				(font
+					(size 1.27 1.27)
+				)
+			)
+		)
+		(property "Field6" "nf"
+			(at 43.18 171.45 0)
+			(hide yes)
+			(show_name no)
+			(do_not_autoplace no)
+			(effects
+				(font
+					(size 1.27 1.27)
+				)
+			)
+		)
+		(property "Field7" "nf"
+			(at 43.18 171.45 0)
+			(hide yes)
+			(show_name no)
+			(do_not_autoplace no)
+			(effects
+				(font
+					(size 1.27 1.27)
+				)
+			)
+		)
+		(property "Part Description" "M2.5 mounting hole"
+			(at 43.18 171.45 0)
+			(hide yes)
+			(show_name no)
+			(do_not_autoplace no)
+			(effects
+				(font
+					(size 1.27 1.27)
+				)
+			)
+		)
+		(instances
+			(project "CM5IO"
+				(path "/e63e39d7-6ac0-4ffd-8aa3-1841a4541b55"
+					(reference "H6")
+					(unit 1)
+				)

Commit message: Updated KiCad files
Parts:
- removed H7, H8: MountingHole, CM5IO:MountingHole_2.7mm_M2.5_DIN965, symbol Mechanical:MountingHole

Commit message: Update BuggyBot KiCad project
Parts:
- added H7: MountingHole, CM5IO:MountingHole_2.7mm_M2.5_DIN965, symbol Mechanical:MountingHole
Changed lines of the file:
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@@
+	)
+	(symbol
+		(lib_id "Mechanical:MountingHole")
+		(at 43.18 176.53 0)
+		(unit 1)
+		(body_style 1)
+		(exclude_from_sim yes)
+		(in_bom no)
+		(on_board yes)
+		(in_pos_files yes)
+		(dnp yes)
+		(property "Reference" "H7"
+			(at 45.72 175.387 0)
+			(show_name no)
+			(do_not_autoplace no)
+			(effects
+				(font
+					(size 1.27 1.27)
+				)
+				(justify left)
+			)
+		)
+		(property "Value" "MountingHole"
+			(at 45.72 177.673 0)
+			(show_name no)
+			(do_not_autoplace no)
+			(effects
+				(font
+					(size 1.27 1.27)
+				)
+				(justify left)
+			)
+		)
+		(property "Footprint" "CM5IO:MountingHole_2.7mm_M2.5_DIN965"
+			(at 43.18 176.53 0)
+			(hide yes)
+			(show_name no)
+			(do_not_autoplace no)
+			(effects
+				(font
+					(size 1.27 1.27)
+				)
+			)
+		)
+		(property "Datasheet" ""
+			(at 43.18 176.53 0)
+			(hide yes)
+			(show_name no)
+			(do_not_autoplace no)
+			(effects
+				(font
+					(size 1.27 1.27)
+				)
+			)
+		)
+		(property "Description" ""
+			(at 43.18 176.53 0)
+			(hide yes)
+			(show_name no)
+			(do_not_autoplace no)
+			(effects
+				(font
+					(size 1.27 1.27)
+				)
+			)
+		)
+		(property "Field4" "nf"
+			(at 43.18 176.53 0)
+			(hide yes)
+			(show_name no)
+			(do_not_autoplace no)
+			(effects
+				(font
+					(size 1.27 1.27)
+				)
+			)
+		)
+		(property "Field5" "nf"
+			(at 43.18 176.53 0)
+			(hide yes)
+			(show_name no)
+			(do_not_autoplace no)
+			(effects
+				(font
+					(size 1.27 1.27)
+				)
+			)
+		)
+		(property "Field6" "nf"
+			(at 43.18 176.53 0)
+			(hide yes)
+			(show_name no)
+			(do_not_autoplace no)
+			(effects
+				(font
+					(size 1.27 1.27)
+				)
+			)
+		)
+		(property "Field7" "nf"
+			(at 43.18 176.53 0)
+			(hide yes)
+			(show_name no)
+			(do_not_autoplace no)
+			(effects
+				(font
+					(size 1.27 1.27)
+				)
+			)
+		)
+		(property "Part Description" "M2.5 mounting hole"
+			(at 43.18 176.53 0)
+			(hide yes)
+			(show_name no)
+			(do_not_autoplace no)
+			(effects
+				(font
+					(size 1.27 1.27)
+				)
+			)
+		)
+		(instances
+			(project "CM5IO"
+				(path "/e63e39d7-6ac0-4ffd-8aa3-1841a4541b55"
+					(reference "H7")
+					(unit 1)
+				)
+			)
+		)
 	)
 	(symbol
